File: resistor_switch.kicad_sch (KiCad schematic)
At the start: 3 parts, among them SW1 SW_SP4T_NR01104

Commit message: move it again
Other:
- moved on the sheet: RN1
Changed lines of the file:
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@@
   (junction (at 100.33 95.25) (diameter 1.016) (color 0 0 0 0)
   )
-  (wire (pts (xy 125.73 74.295) (xy 125.72999 95.25))
+  (wire (pts (xy 139.065 69.215) (xy 139.06499 95.25))
     (stroke (width 0) (type default))
   )
-  (wire (pts (xy 78.74 78.74) (xy 78.74 64.13501))
+  (wire (pts (xy 78.74 78.74) (xy 78.74 59.05501))
     (stroke (width 0) (type default))
   )
@@
     (stroke (width 0) (type default))
   )
-  (wire (pts (xy 125.72999 95.25) (xy 100.33 95.25))
+  (wire (pts (xy 139.06499 95.25) (xy 100.33 95.25))
     (stroke (width 0) (type default))
   )
@@
     (stroke (width 0) (type default))
   )
-  (wire (pts (xy 78.74 64.13501) (xy 118.11 64.135))
+  (wire (pts (xy 78.74 59.05501) (xy 131.445 59.055))
     (stroke (width 0) (type default))
   )
@@
     (fields_autoplaced yes)
   )
-  (symbol (lib_id "Device:R_Network04") (at 123.19 69.215 0) (unit 1)
+  (symbol (lib_id "Device:R_Network04") (at 136.525 64.135 0) (unit 1)
     (in_bom yes) (on_board yes) (exclude_from_sim no) (dnp no)
-    (property "Reference" "RN1" (at 128.27 68.1989 0)
+    (property "Reference" "RN1" (at 141.605 63.1189 0)
       (effects (font (size 1.27 1.27)) (justify left))
     )
-    (property "Value" "R_Network04" (at 128.27 70.7389 0)
+    (property "Value" "R_Network04" (at 141.605 65.6589 0)
       (effects (font (size 1.27 1.27)) (justify left))
     )
-    (property "Footprint" "Resistor_THT:R_Array_SIP5" (at 130.175 69.215 90)
+    (property "Footprint" "Resistor_THT:R_Array_SIP5" (at 143.51 64.135 90)
       (effects (font (size 1.27 1.27)) (hide yes))
     )
-    (property "Datasheet" "http://www.vishay.com/docs/31509/csc.pdf" (at 123.19 69.215 0)
+    (property "Datasheet" "http://www.vishay.com/docs/31509/csc.pdf" (at 136.525 64.135 0)
       (effects (font (size 1.27 1.27)) (hide yes))
     )
-    (property "Description" "4 resistor network, star topology, bussed resistors, small symbol" (at 123.19 69.215 0)
+    (property "Description" "4 resistor network, star topology, bussed resistors, small symbol" (at 136.525 64.135 0)
       (effects (font (size 1.27 1.27)) (hide yes))
     )
