File: test-doc-3c427992.kicad_sch (KiCad schematic)
At the start: 0 parts

Commit message: add some stuff
Parts:
- added U1: AD40xxBCPZ, Package_CSP:LFCSP-WD-10-1EP_3x3mm_P0.5mm_EP1.64x2.38mm, symbol Analog_ADC:AD40xxBCPZ
Changed lines of the file:
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@@
   (title_block
   )
+  (symbol (lib_id "Analog_ADC:AD40xxBCPZ") (at 123.825 90.17 0) (unit 1)
+    (in_bom yes) (on_board yes) (exclude_from_sim no) (dnp no)
+    (property "Reference" "U1" (at 129.883384 78.746048 0)
+      (effects (font (size 1.27 1.27)))
+    )
+    (property "Value" "AD40xxBCPZ" (at 134.54005 80.940124 0)
+      (effects (font (size 1.27 1.27)))
+    )
+    (property "Footprint" "Package_CSP:LFCSP-WD-10-1EP_3x3mm_P0.5mm_EP1.64x2.38mm" (at 123.825 110.49 0)
+      (effects (font (size 1.27 1.27)) (hide yes))
+    )
+    (property "Datasheet" "https://www.analog.com/media/en/technical-documentation/data-sheets/ad4003-4007-4011.pdf" (at 123.825 113.030001 0)
+      (effects (font (size 1.27 1.27)) (hide yes))
+    )
+    (property "Description" "18-Bit, 2 MSPS/1 MSPS/500 kSPS, Differential SAR ADCs, 2.4V to 5.1V reference, 1.8V supply, 1.71 to 5.5V logic IO, 3x3mm LFCSP-10" (at 123.825 90.17 0)
+      (effects (font (size 1.27 1.27)) (hide yes))
+    )
+    (property "ki_keywords" "ADC 18-bit AD4003BCPZ AD4007BCPZ AD4011BCPZ" (at 123.825 90.17 0)
+      (effects (font (size 1.27 1.27)) (hide yes))
+    )
+    (property "ki_fp_filters" "*LFCSP?WD*EP?3x3mm?P0.5mm?EP1.64x2.38mm*" (at 123.825 90.17 0)
+      (effects (font (size 1.27 1.27)) (hide yes))
+    )
+    (pin "1")
+    (pin "10")
+    (pin "11")
+    (pin "2")
+    (pin "3")
+    (pin "4")
+    (pin "5")
+    (pin "6")
+    (pin "7")
+    (pin "8")
+    (pin "9")
+    (instances
+      (project "unknown"
+        (path "/669d2ef9-82a3-4897-8c83-80409d2429ba"
+          (reference "U1") (unit 1)
+        )
+      )
+    )
+    (fields_autoplaced yes)
+  )
 )
