File: test-doc-1769199094607-q4jfu272.kicad_sch (KiCad schematic)
At the start: 0 parts

Commit message: add symbol
Parts:
- added U1: 74AHC240, symbol 74xx:74AHC240
Changed lines of the file:
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@@
   (title_block
   )
+  (symbol (lib_name "74AHC240_1") (lib_id "74xx:74AHC240") (at 110.624387 65.902593 0) (unit 1)
+    (in_bom yes) (on_board yes) (exclude_from_sim no) (dnp no)
+    (property "Reference" "U1" (at 112.575349 47.389017 0)
+      (effects (font (size 1.27 1.27)) (justify left))
+    )
+    (property "Value" "74AHC240" (at 112.575349 49.222655 0)
+      (effects (font (size 1.27 1.27)) (justify left))
+    )
+    (property "Footprint" "" (at 110.624387 65.902593 0)
+      (effects (font (size 1.27 1.27)) (hide yes))
+    )
+    (property "Datasheet" "https://www.ti.com/lit/ds/symlink/sn54ahc240.pdf" (at 110.624387 65.902593 0)
+      (effects (font (size 1.27 1.27)) (hide yes))
+    )
+    (property "Description" "8-bit Buffer/Line Driver 3-state Inverting" (at 110.624387 65.902593 0)
+      (effects (font (size 1.27 1.27)) (hide yes))
+    )
+    (property "ki_keywords" "AHCMOS BUFFER 3State inv" (at 110.624387 65.902593 0)
+      (effects (font (size 1.27 1.27)) (hide yes))
+    )
+    (property "ki_fp_filters" "DIP*W7.62mm* SOIC*7.5x12.8mm*P1.27mm* TSSOP*4.4x6.5mm*P0.65mm* SSOP*4.4x6.5mm*P0.65mm*" (at 110.624387 65.902593 0)
+      (effects (font (size 1.27 1.27)) (hide yes))
+    )
+    (pin "2")
+    (pin "4")
+    (pin "6")
+    (pin "8")
+    (pin "17")
+    (pin "15")
+    (pin "13")
+    (pin "11")
+    (pin "1")
+    (pin "19")
+    (pin "20")
+    (pin "10")
+    (pin "18")
+    (pin "16")
+    (pin "14")
+    (pin "12")
+    (pin "3")
+    (pin "5")
+    (pin "7")
+    (pin "9")
+    (instances
+      (project "unknown"
+        (path "/9a3460b3-3ea5-4782-a0b5-5870fc806a11"
+          (reference "U1") (unit 1)
+        )
+      )
+    )
+    (fields_autoplaced yes)
+  )
 )
