File: test-doc-1769199094607-q4jfu272.kicad_sch (KiCad schematic)
At the start: 0 parts

Commit message: boop boop
Parts:
- added U1: 74HC237, symbol 74xx_IEEE:74HC237
Changed lines of the file:
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@@
   (title_block
   )
+  (symbol (lib_id "74xx_IEEE:74HC237") (at 74.396104 71.447403 0) (unit 1)
+    (in_bom yes) (on_board yes) (exclude_from_sim no) (dnp no)
+    (property "Reference" "U1" (at 76.347066 52.933827 0)
+      (effects (font (size 1.27 1.27)) (justify left))
+    )
+    (property "Value" "74HC237" (at 76.347066 54.767465 0)
+      (effects (font (size 1.27 1.27)) (justify left))
+    )
+    (property "Footprint" "" (at 74.396104 71.447403 0)
+      (effects (font (size 1.27 1.27)) (hide yes))
+    )
+    (property "Datasheet" "" (at 74.396104 71.447403 0)
+      (effects (font (size 1.27 1.27)) (hide yes))
+    )
+    (property "Description" "" (at 74.396104 71.447403 0)
+      (effects (font (size 1.27 1.27)) (hide yes))
+    )
+    (pin "16")
+    (pin "8")
+    (pin "4")
+    (pin "5")
+    (pin "6")
+    (pin "1")
+    (pin "2")
+    (pin "3")
+    (pin "15")
+    (pin "14")
+    (pin "13")
+    (pin "12")
+    (pin "11")
+    (pin "10")
+    (pin "9")
+    (pin "7")
+    (instances
+      (project "unknown"
+        (path "/9a3460b3-3ea5-4782-a0b5-5870fc806a11"
+          (reference "U1") (unit 1)
+        )
+      )
+    )
+    (fields_autoplaced yes)
+  )
 )
